File: Kicad/Projet_Kicad/My_gaz_sensor/My_gaz_sensor.sch (KiCad schematic (older format))
At the start: 21 parts, among them P1 Power, P2 Analog, P3 Digital, P4 Digital, P5 CONN_01X01, P6 CONN_01X01, P7 CONN_01X01, P8 CONN_01X01, U1 LTC1050, U11 RN2483A

Commit message: Refactor valeur C4
Parts:
- C4: value 100n -> 1μ
- U1: symbol MyLib:LTC1050 -> My_gaz_sensor-rescue:LTC1050-MyLib
Changed lines of the file:
@@
 P 6000 3150
 F 0 "C4" H 6115 3196 50  0000 L CNN
-F 1 "100n" H 6115 3105 50  0000 L CNN
+F 1 "1μ" H 6115 3105 50  0000 L CNN
 F 2 "Capacitor_THT:C_Radial_D4.0mm_H5.0mm_P1.50mm" H 6038 3000 50  0001 C CNN
 F 3 "~" H 6000 3150 50  0001 C CNN
@@
 $EndComp
 $Comp
-L MyLib:LTC1050 U1
+L My_gaz_sensor-rescue:LTC1050-MyLib U1
 U 1 1 5E1F5F5E
 P 5150 2800
@@
 $EndComp
 $Comp
-L power:PWR_FLAG #FLG?
+L power:PWR_FLAG #FLG0101
 U 1 1 5E1E5C42
 P 5150 1350
-F 0 "#FLG?" H 5150 1425 50  0001 C CNN
+F 0 "#FLG0101" H 5150 1425 50  0001 C CNN
 F 1 "PWR_FLAG" H 5150 1523 50  0000 C CNN
 F 2 "" H 5150 1350 50  0001 C CNN
@@
 $EndComp
 $Comp
-L power:PWR_FLAG #FLG?
+L power:PWR_FLAG #FLG0102
 U 1 1 5E1E5F87
 P 5600 1350
-F 0 "#FLG?" H 5600 1425 50  0001 C CNN
+F 0 "#FLG0102" H 5600 1425 50  0001 C CNN
 F 1 "PWR_FLAG" H 5600 1523 50  0000 C CNN
 F 2 "" H 5600 1350 50  0001 C CNN
@@
 $EndComp
 $Comp
-L power:PWR_FLAG #FLG?
+L power:PWR_FLAG #FLG0103
 U 1 1 5E1E9BAC
 P 5900 1350
-F 0 "#FLG?" H 5900 1425 50  0001 C CNN
+F 0 "#FLG0103" H 5900 1425 50  0001 C CNN
 F 1 "PWR_FLAG" H 5900 1523 50  0000 C CNN
 F 2 "" H 5900 1350 50  0001 C CNN
