File: Kicad/Projet_Kicad_Aime_plan_masse/My_gaz_sensor/My_gaz_sensor.sch (KiCad schematic (older format))
At the start: 23 parts, among them J1 Conn_01x03, J2 Conn_01x03, P1 Power, P2 Analog, P3 Digital, P4 Digital, P5 CONN_01X01, P6 CONN_01X01, P7 CONN_01X01, P8 CONN_01X01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

Commit message: Refactor valeur C4
Parts:
- C4: value 100n -> 1µ
Other:
- moved on the sheet: J1, J2, S11
Changed lines of the file:
@@
 P 6000 3150
 F 0 "C4" H 6115 3196 50  0000 L CNN
-F 1 "100n" H 6115 3105 50  0000 L CNN
+F 1 "1µ" H 6115 3105 50  0000 L CNN
 F 2 "Capacitor_THT:C_Radial_D4.0mm_H5.0mm_P1.50mm" H 6038 3000 50  0001 C CNN
 F 3 "~" H 6000 3150 50  0001 C CNN
@@
 L power:GND #PWR06
 U 1 1 5E1CB4FB
-P 2650 2500
-F 0 "#PWR06" H 2650 2250 50  0001 C CNN
-F 1 "GND" H 2655 2327 50  0000 C CNN
-F 2 "" H 2650 2500 50  0001 C CNN
-F 3 "" H 2650 2500 50  0001 C CNN
-	1    2650 2500
+P 2750 1600
+F 0 "#PWR06" H 2750 1350 50  0001 C CNN
+F 1 "GND" H 2755 1427 50  0000 C CNN
+F 2 "" H 2750 1600 50  0001 C CNN
+F 3 "" H 2750 1600 50  0001 C CNN
+	1    2750 1600
 	0    -1   -1   0
 $EndComp
@@
 $EndComp
 Wire Wire Line
-	2500 2500 2650 2500
+	2600 1600 2750 1600
 Wire Wire Line
 	4050 3000 4050 3100
@@
 L MyLib:Gaz_Sensor S11
 U 1 1 5E2725E8
-P 1750 2200
-F 0 "S11" H 1700 2415 50  0000 C CNN
-F 1 "Gaz_Sensor" H 1700 2324 50  0000 C CNN
-F 2 "Package_TO_SOT_THT:TO-5-10_Window" H 1400 2400 50  0001 C CNN
-F 3 "" H 1400 2400 50  0001 C CNN
-	1    1750 2200
+P 1850 1300
+F 0 "S11" H 1800 1515 50  0000 C CNN
+F 1 "Gaz_Sensor" H 1800 1424 50  0000 C CNN
+F 2 "Package_TO_SOT_THT:TO-5-10_Window" H 1500 1500 50  0001 C CNN
+F 3 "" H 1500 1500 50  0001 C CNN
+	1    1850 1300
 	1    0    0    -1
 $EndComp
@@
 L Connector_Generic:Conn_01x03 J2
 U 1 1 5E276475
-P 2250 4650
-F 0 "J2" V 2214 4462 50  0000 R CNN
-F 1 "Conn_01x03" V 2123 4462 50  0000 R CNN
-F 2 "Connector_PinHeader_2.00mm:PinHeader_1x03_P2.00mm_Vertical" H 2250 4650 50  0001 C CNN
-F 3 "~" H 2250 4650 50  0001 C CNN
-	1    2250 4650
+P 2350 3750
+F 0 "J2" V 2314 3562 50  0000 R CNN
+F 1 "Conn_01x03" V 2223 3562 50  0000 R CNN
+F 2 "Connector_PinHeader_2.00mm:PinHeader_1x03_P2.00mm_Vertical" H 2350 3750 50  0001 C CNN
+F 3 "~" H 2350 3750 50  0001 C CNN
+	1    2350 3750
 	0    -1   -1   0
 $EndComp
@@
 L Connector_Generic:Conn_01x03 J1
 U 1 1 5E27739D
-P 2250 4450
-F 0 "J1" V 2122 4630 50  0000 L CNN
-F 1 "Conn_01x03" V 2213 4630 50  0000 L CNN
-F 2 "Connector_PinHeader_2.00mm:PinHeader_1x03_P2.00mm_Vertical" H 2250 4450 50  0001 C CNN
-F 3 "~" H 2250 4450 50  0001 C CNN
-	1    2250 4450
+P 2350 3550
+F 0 "J1" V 2222 3730 50  0000 L CNN
+F 1 "Conn_01x03" V 2313 3730 50  0000 L CNN
+F 2 "Connector_PinHeader_2.00mm:PinHeader_1x03_P2.00mm_Vertical" H 2350 3550 50  0001 C CNN
+F 3 "~" H 2350 3550 50  0001 C CNN
+	1    2350 3550
 	0    1    1    0
 $EndComp
 Wire Wire Line
-	2350 4250 2350 4150
-Wire Wire Line
-	2350 4150 2600 4150
-Wire Wire Line
-	2250 4250 2250 4050
-Wire Wire Line
-	2250 4050 2600 4050
-Wire Wire Line
-	2150 4250 2150 3950
-Wire Wire Line
-	2150 3950 2600 3950
-Wire Wire Line
-	2350 4850 2350 5000
-Wire Wire Line
-	2350 5000 2650 5000
-Wire Wire Line
-	2250 4850 2250 5150
-Wire Wire Line
-	2250 5150 2650 5150
-Wire Wire Line
-	2150 4850 2150 5300
-Wire Wire Line
-	2150 5300 2650 5300
+	2450 3350 2450 3250
+Wire Wire Line
+	2450 3250 2700 3250
+Wire Wire Line
+	2350 3350 2350 3150
+Wire Wire Line
+	2350 3150 2700 3150
+Wire Wire Line
+	2250 3350 2250 3050
+Wire Wire Line
+	2250 3050 2700 3050
+Wire Wire Line
+	2450 3950 2450 4100
+Wire Wire Line
+	2450 4100 2750 4100
+Wire Wire Line
+	2350 3950 2350 4250
+Wire Wire Line
+	2350 4250 2750 4250
+Wire Wire Line
+	2250 3950 2250 4400
+Wire Wire Line
+	2250 4400 2750 4400
 $Comp
 L power:+5V #PWR017
 U 1 1 5E29310B
-P 2750 2000
-F 0 "#PWR017" H 2750 1850 50  0001 C CNN
-F 1 "+5V" H 2765 2173 50  0000 C CNN
-F 2 "" H 2750 2000 50  0001 C CNN
-F 3 "" H 2750 2000 50  0001 C CNN
-	1    2750 2000
+P 2850 1100
+F 0 "#PWR017" H 2850 950 50  0001 C CNN
+F 1 "+5V" H 2865 1273 50  0000 C CNN
+F 2 "" H 2850 1100 50  0001 C CNN
+F 3 "" H 2850 1100 50  0001 C CNN
+	1    2850 1100
 	1    0    0    -1
 $EndComp
@@
 L power:GND #PWR016
 U 1 1 5E29549B
-P 2650 3250
-F 0 "#PWR016" H 2650 3000 50  0001 C CNN
-F 1 "GND" H 2655 3077 50  0000 C CNN
-F 2 "" H 2650 3250 50  0001 C CNN
-F 3 "" H 2650 3250 50  0001 C CNN
-	1    2650 3250
+P 2750 2350
+F 0 "#PWR016" H 2750 2100 50  0001 C CNN
+F 1 "GND" H 2755 2177 50  0000 C CNN
+F 2 "" H 2750 2350 50  0001 C CNN
+F 3 "" H 2750 2350 50  0001 C CNN
+	1    2750 2350
 	0    -1   -1   0
 $EndComp
 Wire Wire Line
-	2500 3150 2500 3250
-Wire Wire Line
-	2500 3250 2650 3250
-Connection ~ 2500 3250
-Wire Wire Line
-	2500 3250 2500 3350
-Wire Wire Line
-	2500 2300 2750 2300
-Wire Wire Line
-	2750 2300 2750 2000
-Wire Wire Line
-	2500 2750 2900 2750
-Wire Wire Line
-	2500 2950 2900 2950
-Wire Wire Line
-	900  2750 600  2750
-Wire Wire Line
-	900  2950 600  2950
-NoConn ~ 900  2300
-NoConn ~ 900  2500
-Text Label 600  2750 0    50   ~ 0
+	2600 2250 2600 2350
+Wire Wire Line
+	2600 2350 2750 2350
+Connection ~ 2600 2350
+Wire Wire Line
+	2600 2350 2600 2450
+Wire Wire Line
+	2600 1400 2850 1400
+Wire Wire Line
+	2850 1400 2850 1100
+Wire Wire Line
+	2600 1850 3000 1850
+Wire Wire Line
+	2600 2050 3000 2050
+Wire Wire Line
+	1000 1850 700  1850
+Wire Wire Line
+	1000 2050 700  2050
+NoConn ~ 1000 1400
+NoConn ~ 1000 1600
+Text Label 700  1850 0    50   ~ 0
 GazSensorLeft1
-Text Label 600  2950 0    50   ~ 0
+Text Label 700  2050 0    50   ~ 0
 GazSensorLeft2
-Text Label 2900 2750 2    50   ~ 0
+Text Label 3000 1850 2    50   ~ 0
 GazSensorRight1
-Text Label 2900 2950 2    50   ~ 0
+Text Label 3000 2050 2    50   ~ 0
 GazSensorRight2
-Text Label 2600 4150 2    50   ~ 0
+Text Label 2700 3250 2    50   ~ 0
 GazSensorRight1
-Text Label 2600 3950 2    50   ~ 0
+Text Label 2700 3050 2    50   ~ 0
 GazSensorLeft1
-Text Label 2650 5000 2    50   ~ 0
+Text Label 2750 4100 2    50   ~ 0
 GazSensorRight2
-Text Label 2650 5300 2    50   ~ 0
+Text Label 2750 4400 2    50   ~ 0
 GazSensorLeft2
 $Comp
 L power:+5V #PWR05
 U 1 1 5E2D70AD
-P 2650 5150
-F 0 "#PWR05" H 2650 5000 50  0001 C CNN
-F 1 "+5V" V 2665 5278 50  0000 L CNN
-F 2 "" H 2650 5150 50  0001 C CNN
-F 3 "" H 2650 5150 50  0001 C CNN
-	1    2650 5150
+P 2750 4250
+F 0 "#PWR05" H 2750 4100 50  0001 C CNN
+F 1 "+5V" V 2765 4378 50  0000 L CNN
+F 2 "" H 2750 4250 50  0001 C CNN
+F 3 "" H 2750 4250 50  0001 C CNN
+	1    2750 4250
 	0    1    1    0
 $EndComp
-Text Label 2600 4050 2    50   ~ 0
+Text Label 2700 3150 2    50   ~ 0
 link_circuit
 $Comp
