File: Kicad/Projet_Kicad_Aime_plan_masse/My_gaz_sensor/My_gaz_sensor.sch (KiCad schematic (older format))
At the start: 24 parts, among them J1 Conn_01x03, J2 Conn_01x03, P1 Power, P2 Analog, P3 Digital, P4 Digital, P5 CONN_01X01, P6 CONN_01X01, P7 CONN_01X01, P8 CONN_01X01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

Commit message: Refactor Aime Kicad Part
Parts:
- U1: footprint MyComponent:PDIP-8_N -> Package_DIP:DIP-8_W7.62mm_LongPads
Changed lines of the file:
@@
 F 0 "U1" H 5544 2971 50  0000 L CNN
 F 1 "LTC1050" H 5544 2880 50  0000 L CNN
-F 2 "MyComponent:PDIP-8_N" H 5450 3100 50  0001 C CNN
+F 2 "Package_DIP:DIP-8_W7.62mm_LongPads" H 5450 3100 50  0001 C CNN
 F 3 "" H 5450 3100 50  0001 C CNN
 	1    5400 2900
