File: Kicad/Projet_Kicad_plan_masse/My_gaz_sensor/My_gaz_sensor.kicad_pcb (KiCad board)
At the start: 2 copper layers, 134.6 x 64.8 mm, 21 parts, among them P1 Power, P2 Analog, P3 Digital, P4 Digital, P5 CONN_01X01, P6 CONN_01X01, P7 CONN_01X01, P8 CONN_01X01, U1 LTC1050, U11 RN2483A

Commit message: Refactor valeur C4
Parts:
- C4: value 100n -> 1μ
Changed lines of the file:
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@@
       (effects (font (size 1 1) (thickness 0.15)))
     )
-    (fp_text value 100n (at 0.75 3.25) (layer F.Fab)
+    (fp_text value 1μ (at 0.75 3.25) (layer F.Fab)
       (effects (font (size 1 1) (thickness 0.15)))
     )
@@
   (segment (start 207.518 83.85) (end 198.15 93.218) (width 0.8) (layer B.Cu) (net 20))
   (segment (start 207.518 80.645) (end 207.518 83.85) (width 0.8) (layer B.Cu) (net 20))
-  (segment (start 142.748 104.775) (end 146.558 100.965) (width 0.8) (layer B.Cu) (net 45))
   (segment (start 146.558 126.365) (end 146.558 123.825) (width 1) (layer B.Cu) (net 28))
   (segment (start 188.468 108.936) (end 188.468 116.205) (width 1) (layer B.Cu) (net 28))
@@
   (segment (start 146.558 84.455) (end 159.258 84.455) (width 0.8) (layer B.Cu) (net 36))
   (segment (start 116.078 103.505) (end 123.698 103.505) (width 0.8) (layer B.Cu) (net 37))
+  (segment (start 142.748 104.775) (end 146.558 100.965) (width 0.8) (layer B.Cu) (net 45))
   (segment (start 149.098 111.125) (end 142.748 104.775) (width 1) (layer B.Cu) (net 45))
   (segment (start 149.098 123.825) (end 149.098 111.125) (width 1) (layer B.Cu) (net 45))
